Commit message: removed manipulator from hw

File: src/zsmall_description/urdf/little_arm.urdf.xacro (robot description, xacro)
@@ -1,3 +1,3 @@
-<?xml version="0.001"?>
+<?xml version="1.0"?>
 <robot xmlns:xacro="http://www.ros.org/wiki/xacro" name="little_arm">
     <!-- Useful XACRO Variables (Properties) -->

File: src/zsmall_description/urdf/smallbot.urdf.xacro (robot description, xacro)
@@ -4,7 +4,10 @@
    <xacro:arg name="is_sim" default="true"/>
    <xacro:arg name="use_ros2_control" default="true"/>
+   <xacro:arg name="use_arm" default="true"/>
   <!-- Include physical aspects of the robot, includes add-ons -->
   <xacro:include filename="$(find zsmall_description)/urdf/smallbot_physical.urdf.xacro" />
-  <xacro:include filename="$(find zsmall_description)/urdf/little_arm.urdf.xacro" />
+  <xacro:if value="$(arg use_arm)">
+      <xacro:include filename="$(find zsmall_description)/urdf/little_arm.urdf.xacro" />
+  </xacro:if>
   <!-- Include ros2 control Parameters for both SIM and REAL robots-->
   <xacro:include filename="$(find zsmall_description)/urdf/smallbot_ros2_control.xacro" />

File: src/zsmall_description/urdf/smallbot_ros2_control.xacro (robot description, xacro)
@@ -41,33 +41,35 @@
             </hardware>
         </xacro:unless>
-        <!-- ros2_control Common Interfaces -->
-        <joint name="joint_1">
-            <command_interface name="position">
-              <param name="min">-1.57</param>
-              <param name="max">1.57</param>
-            </command_interface>
-            <state_interface name="position" />
-        </joint>
-        <joint name="joint_2">
-            <command_interface name="position">
-              <param name="min">-1.57</param>
-              <param name="max">1.57</param>
-            </command_interface>
-            <state_interface name="position" />
-        </joint>
-        <joint name="joint_3">
-            <command_interface name="position">
-              <param name="min">-1.57</param>
-              <param name="max">1.57</param>
-            </command_interface>
-            <state_interface name="position" />
-        </joint>
-        <joint name="joint_4">
-            <command_interface name="position">
-              <param name="min">-1.57</param>
-              <param name="max">0</param>
-            </command_interface>
-            <state_interface name="position" />
-        </joint>
+        <xacro:if value="$(arg use_arm)">
+            <!-- ros2_control Common Interfaces -->
+            <joint name="joint_1">
+                <command_interface name="position">
+                    <param name="min">-1.57</param>
+                    <param name="max">1.57</param>
+                </command_interface>
+                <state_interface name="position" />
+            </joint>
+            <joint name="joint_2">
+                <command_interface name="position">
+                    <param name="min">-1.57</param>
+                    <param name="max">1.57</param>
+                </command_interface>
+                <state_interface name="position" />
+            </joint>
+            <joint name="joint_3">
+                <command_interface name="position">
+                    <param name="min">-1.57</param>
+                    <param name="max">1.57</param>
+                </command_interface>
+                <state_interface name="position" />
+            </joint>
+            <joint name="joint_4">
+                <command_interface name="position">
+                    <param name="min">-1.57</param>
+                    <param name="max">0</param>
+                </command_interface>
+                <state_interface name="position" />
+            </joint>
+        </xacro:if>
     </ros2_control>
 </robot>
