Commit message: matching nav in bigbot except dims

File: src/zsmall_description/urdf/smallbot.urdf.xacro (robot description, xacro)
@@ -4,7 +4,8 @@
    <xacro:arg name="is_sim" default="true"/>
    <xacro:arg name="use_ros2_control" default="true"/>
-   <xacro:arg name="use_arm" default="true"/>
+   <xacro:arg name="use_arm" default="false"/>
   <!-- Include physical aspects of the robot, includes add-ons -->
   <xacro:include filename="$(find zsmall_description)/urdf/smallbot_physical.urdf.xacro" />
+  <xacro:include filename="$(find zsmall_description)/urdf/materials.xacro" />
   <xacro:if value="$(arg use_arm)">
       <xacro:include filename="$(find zsmall_description)/urdf/little_arm.urdf.xacro" />

File: src/zsmall_description/urdf/smallbot_gazebo_control.xacro (robot description, xacro)
@@ -98,5 +98,5 @@
    <!-- 2D Laser Sensor -->
    <gazebo reference="laser_frame">
-    <sensor name="lidar" type="gpu_lidar">
+    <sensor name="gpu_lidar" type="gpu_lidar">
       <always_on>true</always_on>
       <visualize>true</visualize>

File: src/zsmall_description/urdf/smallbot_physical.urdf.xacro (robot description, xacro)
@@ -1,29 +1,32 @@
 <?xml version="1.0"?>
 <robot name="zsmall" xmlns:xacro="http://ros.org/wiki/xacro">
-  <material name="blue">
-    <color rgba="0 0 1 1"/>
-  </material>
-  <material name="black">
-    <color rgba="0 0 0 1"/>
-  </material>
-  <material name="white">
-  <color rgba="1 1 1 1"/>
-  </material>
-  <material name="silver">
-    <color rgba="0.79 0.82 0.93 1"/>
-  </material>
-  <material name="dark_grey">
-    <color rgba="0.3 0.3 0.3 1"/>
-  </material>
-  <link name="base_footprint"/>
+    <xacro:property name="wheel_radius" value="0.033"/>
+    <xacro:property name="wheel_offset_y" value="0.141"/>
+    <xacro:property name="wheel_offset_z" value="0.0225"/>
+    <xacro:property name="caster_wheel_radius" value="0.051"/>
+    <xacro:property name="caster_wheel_offset_x" value="0.137"/>
+    <xacro:property name="caster_wheel_offset_y" value="0.095"/>
+    <xacro:property name="caster_wheel_offset_z" value="0.0133"/>
+    <xacro:property name="imu_roll" value="0.0"/>
+    <xacro:property name="imu_pitch" value="0.0"/>
+    <xacro:property name="imu_yaw" value="1.57"/>
+    <xacro:property name="lidar_roll" value="0.0"/>
+    <xacro:property name="lidar_pitch" value="0.0"/>
+    <xacro:property name="lidar_yaw" value="3.14"/>
+    <xacro:property name="chassis_mass" value="1.409"/>
+    <xacro:property name="wheel_mass" value="0.05"/>
+    <xacro:property name="caster_wheel_mass" value="0.01"/>
+  <!-- BASE_FOOTPRINT LINK -->
+  <link name="base_footprint"></link>
+   <!-- BASE LINK -->
   <link name="base_link">
     <inertial>
       <origin xyz="-0.070489 -0.000718 0.040699" rpy="0.0 0.0 0.0" />
-      <mass value="1.409448"/>
+      <mass value="${chassis_mass}"/>
       <inertia ixx="0.011114" ixy="0.000188" ixz="-0.005821"
                iyy="0.017229" iyz="0.000127"
                izz="0.019734" />
     </inertial>
-    <visual>
+    <visual name='base_link_visual'>
       <origin xyz="0 0 0" rpy="0 0 0" />
       <geometry>
@@ -39,13 +42,14 @@
     </collision>
   </link>
-  <joint name="base_joint" type="fixed">
+   <joint name="base_joint" type="fixed">
     <parent link="base_footprint"/>
     <child link="base_link" />
-    <origin xyz="0 0 0.033" rpy="0 0 0"/>
-  </joint>
+    <origin xyz="0 0 ${wheel_radius}" rpy="0 0 0"/>
+  </joint>
+<!-- RIGHT WHEEL LINK -->
   <link name="wheel_right_link">
     <inertial>
       <origin xyz="0 -0.014 0" rpy="0 0 0" />
-      <mass value="0.0530086090966721" />
+      <mass value="${wheel_mass}" />
       <inertia ixx="1.88176298336665E-05" ixy="-4.8444933029987E-10" ixz="1.88163708851143E-08"
                iyy="3.11510738647764E-05" iyz="-6.93560663069607E-11"
@@ -62,19 +66,20 @@
       <origin xyz="0 -0.015 0" rpy="1.57 0 0" />
       <geometry>
-        <sphere radius="0.033"/>
+        <sphere radius="${wheel_radius}"/>
       </geometry>
     </collision>
   </link>
   <joint name="wheel_right_joint" type="continuous">
-    <origin xyz="0 -0.141 0" rpy="0 0 0" />
+    <origin xyz="0 ${-wheel_offset_y} 0" rpy="0 0 0" />
     <parent link="base_link" />
     <child link="wheel_right_link" />
     <axis xyz="0 1 0" />
   </joint>
+<!-- LEFT WHEEL LINK -->
   <link
     name="wheel_left_link">
     <inertial>
       <origin xyz="0 -0.014 0" rpy="0 0 0" />
-      <mass value="0.0530086043217644" />
+      <mass value="${wheel_mass}" />
       <inertia ixx="1.8792911368909E-05"  ixy="3.31256392204584E-10" ixz="-1.14082001662767E-08"
                iyy="3.11510738759073E-05" iyz="-3.60499245082192E-10"
@@ -91,14 +96,15 @@
       <origin xyz="0 -0.014 0" rpy="-1.57 0 0" />
       <geometry>
-        <sphere radius="0.033"/>
+        <sphere radius="${wheel_radius}"/>
       </geometry>
     </collision>
   </link>
   <joint name="wheel_left_joint" type="continuous">
-    <origin xyz="0 0.141 0" rpy="0 0 0" />
+    <origin xyz="0 ${wheel_offset_y}  0" rpy="0 0 0" />
     <parent link="base_link" />
     <child link="wheel_left_link" />
     <axis xyz="0 1 0" />
   </joint>
+<!-- RIGHT CASTER WHEEL LINK -->
   <link name="caster_right_link">
     <inertial>
@@ -119,14 +125,15 @@
       <origin xyz="0 0 0" rpy="0 0 0" />
       <geometry>
-        <sphere radius="0.051"/>
+        <sphere radius="${wheel_radius}"/>
       </geometry>
     </collision>
   </link>
   <joint name="caster_right_joint" type="fixed">
-    <origin xyz="-0.137 -0.095 .0133" rpy="1.57 0 1.57" />
+    <origin xyz="${-caster_wheel_offset_x} ${-caster_wheel_offset_y} ${-caster_wheel_offset_z}" rpy="1.57 0 1.57" />
     <parent link="base_link" />
     <child link="caster_right_link" />
     <axis xyz="0 0 0" />
   </joint>
+<!-- LEFT CASTER WHEEL LINK -->
   <link name="caster_left_link">
     <inertial>
@@ -147,14 +154,15 @@
       <origin xyz="0 0 0" rpy="0 0 0" />
       <geometry>
-        <sphere radius="0.051"/>
+        <sphere radius="${wheel_radius}"/>
       </geometry>
     </collision>
   </link>
   <joint name="caster_left_joint" type="fixed">
-    <origin xyz="-0.137 0.095 0.0133" rpy="1.57 0 1.57" />
+    <origin xyz="${-caster_wheel_offset_x} ${caster_wheel_offset_y} ${-caster_wheel_offset_z}" rpy="1.57 0 1.57" />
     <parent link="base_link" />
     <child link="caster_left_link" />
     <axis xyz="0 0 0" />
   </joint>
+<!-- IMU LINK -->
   <link name="imu_link">
     <inertial>
@@ -173,5 +181,5 @@
     </visual>
     <collision>
-      <origin xyz="0 0 0" rpy="0 0 1.57" />
+      <origin xyz="0 0 0" rpy="${imu_roll} ${imu_pitch} ${imu_yaw}" />
       <geometry>
         <mesh filename="file://$(find zsmall_description)/meshes/imu_link.STL" />
@@ -180,9 +188,10 @@
   </link>
   <joint name="imu_joint" type="fixed">
-    <origin xyz="-0.04016 0.049755 0.064953" rpy="3.14 0 -1.57" />
+    <origin xyz="-0.04016 0.049755 0.064953" rpy="${imu_roll} ${imu_pitch} ${imu_yaw}" />
     <parent link="base_link" />
     <child link="imu_link" />
     <axis xyz="0 0 0" />
   </joint>
+<!-- LIDAR LINK -->
   <link name="laser_frame">
     <inertial>
@@ -201,5 +210,5 @@
     </visual>
     <collision>
-      <origin xyz="0 0 0" rpy="0 0 0" />
+      <origin xyz="0 0 0" rpy="${lidar_roll} ${lidar_pitch} ${lidar_yaw}" />
       <geometry>
         <mesh filename="file://$(find zsmall_description)/meshes/lidarA1M8.stl" />
@@ -208,5 +217,5 @@
   </link>
   <joint name="laser_joint" type="fixed">
-    <origin xyz="-0.013456 0.000513 0.140452" rpy="0 0 3.14" />
+    <origin xyz="-0.013456 0.000513 0.140452" rpy="${lidar_roll} ${lidar_pitch} ${lidar_yaw}" />
     <parent link="base_link" />
     <child link="laser_frame" />

Commit message: fixes for urdf experiment

File: src/zsmall_description/urdf/smallbot.urdf.xacro (robot description, xacro)
@@ -7,5 +7,5 @@
   <!-- Include physical aspects of the robot, includes add-ons -->
   <xacro:include filename="$(find zsmall_description)/urdf/smallbot_physical.urdf.xacro" />
-  <xacro:include filename="$(find zsmall_description)/urdf/materials.xacro" />
+  <!-- <xacro:include filename="$(find zsmall_description)/urdf/materials.xacro" /> -->
   <xacro:if value="$(arg use_arm)">
       <xacro:include filename="$(find zsmall_description)/urdf/little_arm.urdf.xacro" />

File: src/zsmall_description/urdf/smallbot_physical.urdf.xacro (robot description, xacro)
@@ -1,4 +1,4 @@
 <?xml version="1.0"?>
-<robot name="mybots" xmlns:xacro="http://ros.org/wiki/xacro">
+<robot name="zsmall" xmlns:xacro="http://ros.org/wiki/xacro">
   <material name="blue">
     <color rgba="0 0 1 1"/>
@@ -28,5 +28,5 @@
       <origin xyz="0 0 0" rpy="0 0 0" />
       <geometry>
-        <mesh filename="file://$(find mybots_description)/meshes/smallbot_base_link.stl" />
+        <mesh filename="file://$(find zsmall_description)/meshes/smallbot_base_link.stl" />
       </geometry>
       <material name="dark_grey"/>
@@ -35,5 +35,5 @@
       <origin xyz="0 0 0" rpy="0 0 0" />
       <geometry>
-        <mesh filename="file://$(find mybots_description)/meshes/smallbot_base_link.stl" />
+        <mesh filename="file://$(find zsmall_description)/meshes/smallbot_base_link.stl" />
       </geometry>
     </collision>
@@ -55,5 +55,5 @@
       <origin xyz="-0.0 0.014 0.0" rpy="1.57 0 0" />
       <geometry>
-        <mesh filename="file://$(find mybots_description)/meshes/smallbot_wheel.stl" />
+        <mesh filename="file://$(find zsmall_description)/meshes/smallbot_wheel.stl" />
       </geometry>
       <material name="blue"/>
@@ -84,5 +84,5 @@
       <origin xyz="0 -0.014 0" rpy="-1.57 0 0" />
       <geometry>
-        <mesh filename="file://$(find mybots_description)/meshes/smallbot_wheel.stl" />
+        <mesh filename="file://$(find zsmall_description)/meshes/smallbot_wheel.stl" />
       </geometry>
       <material name="blue"/>
@@ -112,5 +112,5 @@
       <origin xyz="0 0 0" rpy="0 0 0" />
       <geometry>
-        <mesh filename="file://$(find mybots_description)/meshes/smallbot_caster_link.stl" />
+        <mesh filename="file://$(find zsmall_description)/meshes/smallbot_caster_link.stl" />
       </geometry>
       <material name="silver"/>
@@ -140,5 +140,5 @@
       <origin xyz="0 0 0" rpy="0 0 0" />
       <geometry>
-        <mesh filename="file://$(find mybots_description)/meshes/smallbot_caster_link.stl" />
+        <mesh filename="file://$(find zsmall_description)/meshes/smallbot_caster_link.stl" />
       </geometry>
       <material name="silver"/>
@@ -168,5 +168,5 @@
       <origin xyz="0 0 0" rpy="0 0 3.14" />
       <geometry>
-        <mesh filename="file://$(find mybots_description)/meshes/imu_link.STL" />
+        <mesh filename="file://$(find zsmall_description)/meshes/imu_link.STL" />
       </geometry>
       <material name="blue"/>
@@ -175,5 +175,5 @@
       <origin xyz="0 0 0" rpy="0 0 1.57" />
       <geometry>
-        <mesh filename="file://$(find mybots_description)/meshes/imu_link.STL" />
+        <mesh filename="file://$(find zsmall_description)/meshes/imu_link.STL" />
       </geometry>
     </collision>
@@ -196,5 +196,5 @@
       <origin xyz="0 0 0" rpy="1.57 0 3.14" />
       <geometry>
-        <mesh filename="file://$(find mybots_description)/meshes/lidarA1M8.stl" />
+        <mesh filename="file://$(find zsmall_description)/meshes/lidarA1M8.stl" />
       </geometry>
       <material name="black"/>
@@ -203,5 +203,5 @@
       <origin xyz="0 0 0" rpy="0 0 0" />
       <geometry>
-        <mesh filename="file://$(find mybots_description)/meshes/lidarA1M8.stl" />
+        <mesh filename="file://$(find zsmall_description)/meshes/lidarA1M8.stl" />
       </geometry>
     </collision>

Commit message: Revert "fixes for urdf experiment"
This reverts commit 8e00e7d692f7bab2070bca8851375713b59a609c.

File: src/zsmall_description/urdf/smallbot.urdf.xacro (robot description, xacro)
@@ -7,5 +7,5 @@
   <!-- Include physical aspects of the robot, includes add-ons -->
   <xacro:include filename="$(find zsmall_description)/urdf/smallbot_physical.urdf.xacro" />
-  <!-- <xacro:include filename="$(find zsmall_description)/urdf/materials.xacro" /> -->
+  <xacro:include filename="$(find zsmall_description)/urdf/materials.xacro" />
   <xacro:if value="$(arg use_arm)">
       <xacro:include filename="$(find zsmall_description)/urdf/little_arm.urdf.xacro" />

File: src/zsmall_description/urdf/smallbot_physical.urdf.xacro (robot description, xacro)
@@ -1,4 +1,4 @@
 <?xml version="1.0"?>
-<robot name="zsmall" xmlns:xacro="http://ros.org/wiki/xacro">
+<robot name="mybots" xmlns:xacro="http://ros.org/wiki/xacro">
     <xacro:property name="wheel_radius" value="0.033"/>
     <xacro:property name="wheel_offset_y" value="0.141"/>
@@ -31,5 +31,5 @@
       <origin xyz="0 0 0" rpy="0 0 0" />
       <geometry>
-        <mesh filename="file://$(find zsmall_description)/meshes/smallbot_base_link.stl" />
+        <mesh filename="file://$(find mybots_description)/meshes/smallbot_base_link.stl" />
       </geometry>
       <material name="dark_grey"/>
@@ -38,5 +38,5 @@
       <origin xyz="0 0 0" rpy="0 0 0" />
       <geometry>
-        <mesh filename="file://$(find zsmall_description)/meshes/smallbot_base_link.stl" />
+        <mesh filename="file://$(find mybots_description)/meshes/smallbot_base_link.stl" />
       </geometry>
     </collision>
@@ -59,5 +59,5 @@
       <origin xyz="-0.0 0.014 0.0" rpy="1.57 0 0" />
       <geometry>
-        <mesh filename="file://$(find zsmall_description)/meshes/smallbot_wheel.stl" />
+        <mesh filename="file://$(find mybots_description)/meshes/smallbot_wheel.stl" />
       </geometry>
       <material name="blue"/>
@@ -89,5 +89,5 @@
       <origin xyz="0 -0.014 0" rpy="-1.57 0 0" />
       <geometry>
-        <mesh filename="file://$(find zsmall_description)/meshes/smallbot_wheel.stl" />
+        <mesh filename="file://$(find mybots_description)/meshes/smallbot_wheel.stl" />
       </geometry>
       <material name="blue"/>
@@ -118,5 +118,5 @@
       <origin xyz="0 0.012 0.0" rpy="0 0 0" />
       <geometry>
-        <mesh filename="file://$(find zsmall_description)/meshes/smallbot_caster_link.stl" />
+        <mesh filename="file://$(find mybots_description)/meshes/smallbot_caster_link.stl" />
       </geometry>
       <material name="silver"/>
@@ -147,5 +147,5 @@
       <origin xyz="0 0.012 0" rpy="0 0 0" />
       <geometry>
-        <mesh filename="file://$(find zsmall_description)/meshes/smallbot_caster_link.stl" />
+        <mesh filename="file://$(find mybots_description)/meshes/smallbot_caster_link.stl" />
       </geometry>
       <material name="silver"/>
@@ -176,5 +176,5 @@
       <origin xyz="0 0 0" rpy="0 0 3.14" />
       <geometry>
-        <mesh filename="file://$(find zsmall_description)/meshes/imu_link.STL" />
+        <mesh filename="file://$(find mybots_description)/meshes/imu_link.STL" />
       </geometry>
       <material name="blue"/>
@@ -183,5 +183,5 @@
       <origin xyz="0 0 0" rpy="${imu_roll} ${imu_pitch} ${imu_yaw}" />
       <geometry>
-        <mesh filename="file://$(find zsmall_description)/meshes/imu_link.STL" />
+        <mesh filename="file://$(find mybots_description)/meshes/imu_link.STL" />
       </geometry>
     </collision>
@@ -205,5 +205,5 @@
       <origin xyz="0 0 0" rpy="1.57 0 3.14" />
       <geometry>
-        <mesh filename="file://$(find zsmall_description)/meshes/lidarA1M8.stl" />
+        <mesh filename="file://$(find mybots_description)/meshes/lidarA1M8.stl" />
       </geometry>
       <material name="black"/>
@@ -212,5 +212,5 @@
       <origin xyz="0 0 0" rpy="${lidar_roll} ${lidar_pitch} ${lidar_yaw}" />
       <geometry>
-        <mesh filename="file://$(find zsmall_description)/meshes/lidarA1M8.stl" />
+        <mesh filename="file://$(find mybots_description)/meshes/lidarA1M8.stl" />
       </geometry>
     </collision>
